File: panel meter display rev1/panel meter display rev1.kicad_pcb (KiCad board)
At the start: 2 copper layers, 106.7 x 30.5 mm, 11 parts, among them J1 display

Commit message: gerber zip
Routing:
- net /C2: track 19.4 -> 17.3 mm
Changed lines of the file:
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@@
       (layerselection 0x00010fc_ffffffff)
       (disableapertmacros false)
-      (usegerberextensions false)
+      (usegerberextensions true)
       (usegerberattributes true)
       (usegerberadvancedattributes true)
@@
       (plotinvisibletext false)
       (sketchpadsonfab false)
-      (subtractmaskfromsilk false)
+      (subtractmaskfromsilk true)
       (outputformat 1)
       (mirror false)
-      (drillshape 1)
+      (drillshape 0)
       (scaleselection 1)
-      (outputdirectory "")
+      (outputdirectory "panel meter display rev1-gerbers")
     )
   )
@@
   (segment (start 137.16 40.64) (end 137.16 24.13) (width 0.25) (layer "B.Cu") (net 16))
   (segment (start 134.62 43.18) (end 137.16 40.64) (width 0.25) (layer "B.Cu") (net 16))
-  (segment (start 133.35 34.29) (end 132.08 35.56) (width 0.25) (layer "B.Cu") (net 17))
-  (segment (start 133.387457 25.362543) (end 134.62 24.13) (width 0.25) (layer "B.Cu") (net 17))
-  (segment (start 133.35 38.1) (end 134.62 38.1) (width 0.25) (layer "B.Cu") (net 17))
-  (segment (start 135.544511 32.637054) (end 135.544511 33.402946) (width 0.25) (layer "B.Cu") (net 17))
-  (segment (start 134.638729 31.731271) (end 135.544511 32.637054) (width 0.25) (layer "B.Cu") (net 17))
-  (segment (start 132.08 36.83) (end 133.35 38.1) (width 0.25) (layer "B.Cu") (net 17))
+  (segment (start 135.544511 32.637054) (end 134.638729 31.731271) (width 0.25) (layer "B.Cu") (net 17))
+  (segment (start 134.657457 34.29) (end 135.544511 33.402946) (width 0.25) (layer "B.Cu") (net 17))
   (segment (start 133.387457 30.48) (end 133.387457 25.362543) (width 0.25) (layer "B.Cu") (net 17))
-  (segment (start 132.08 35.56) (end 132.08 36.83) (width 0.25) (layer "B.Cu") (net 17))
+  (segment (start 133.1468 36.6268) (end 133.1468 35.2044) (width 0.25) (layer "B.Cu") (net 17))
+  (segment (start 134.62 38.1) (end 133.1468 36.6268) (width 0.25) (layer "B.Cu") (net 17))
+  (segment (start 134.0612 34.29) (end 134.657457 34.29) (width 0.25) (layer "B.Cu") (net 17))
+  (segment (start 133.1468 35.2044) (end 134.0612 34.29) (width 0.25) (layer "B.Cu") (net 17))
+  (segment (start 135.544511 33.402946) (end 135.544511 32.637054) (width 0.25) (layer "B.Cu") (net 17))
   (segment (start 134.638729 31.731271) (end 133.387457 30.48) (width 0.25) (layer "B.Cu") (net 17))
-  (segment (start 134.657457 34.29) (end 133.35 34.29) (width 0.25) (layer "B.Cu") (net 17))
-  (segment (start 135.544511 33.402946) (end 134.657457 34.29) (width 0.25) (layer "B.Cu") (net 17))
+  (segment (start 133.387457 25.362543) (end 134.62 24.13) (width 0.25) (layer "B.Cu") (net 17))
   (segment (start 136.235489 44.104511) (end 134.237054 44.104511) (width 0.25) (layer "B.Cu") (net 18))
   (segment (start 134.237054 44.104511) (end 133.667859 43.535316) (width 0.25) (layer "B.Cu") (net 18))
